File: docs/e-ink_multi_sensor/e-ink_multi_sensor/e-ink_multi_sensor.kicad_pcb (KiCad board)
At the start: 2 copper layers, 5 parts, among them J1 HC-SR501, J2 SCD41, J3 BME280, U1 ESP32-S3-DevKitC

Commit message: updated schematic
Parts:
- added H1: MountingHole, MountingHole:MountingHole_3mm_Pad, F.Cu at (25.0, 25.5)
- added H2: MountingHole, MountingHole:MountingHole_3mm_Pad, F.Cu at (25.5, 149.5)
- added H3: MountingHole, MountingHole:MountingHole_3mm_Pad, F.Cu at (181.0, 25.0)
- added H4: MountingHole, MountingHole:MountingHole_3mm_Pad, F.Cu at (180.0, 150.0)

Commit message: updated schematic
Parts:
- added J4: WeAct 1, Connector_JST:JST_PH_B8B-PH-K_1x08_P2.00mm_Vertical, F.Cu at (58.5, 73.5)
- added J5: WeAct 2, Connector_Hirose:Hirose_DF11-8DP-2DSA_2x04_P2.00mm_Vertical, F.Cu at (62.0, 91.0)
- moved J2 91.4 mm to (135.0, 107.0)
- moved J3 91.4 mm to (147.5, 107.0)
- moved D1 44.0 mm to (133.6, 77.8)
- moved J1 44.0 mm to (148.5, 77.5)
Connections:
- J2 pad 1: /3v3 -> +3V3
- J3 pad 1: /3v3 -> +3V3
- U1 pad 10: unconnected-(U1-GPIO17/ADC2_CH6-Pad10) -> /SPARE_2
- U1 pad 11: unconnected-(U1-GPIO18/ADC2_CH7-Pad11) -> /SPARE_3
- U1 pad 12: unconnected-(U1-GPIO8/ADC1_CH7-Pad12) -> /WA_CS
- U1 pad 15: unconnected-(U1-GPIO9/ADC1_CH8-Pad15) -> /WA_DC
- U1 pad 16: unconnected-(U1-GPIO10/ADC1_CH9-Pad16) -> /WA_RESET
- U1 pad 17: unconnected-(U1-GPIO11/ADC2_CH0-Pad17) -> /WA_BUSY
- U1 pad 18: /PIR_GPIO12 -> unconnected-(U1-GPIO12/ADC2_CH1-Pad18)
- U1 pad 27: unconnected-(U1-GPIO21-Pad27) -> /SPARE_4
- U1 pad 4: /I2C_SDA -> unconnected-(U1-GPIO4/ADC1_CH3-Pad4)
- U1 pad 5: /I2C_SCL -> unconnected-(U1-GPIO5/ADC1_CH4-Pad5)
- U1 pad 6: unconnected-(U1-GPIO6/ADC1_CH5-Pad6) -> /WA_SCL
- U1 pad 7: unconnected-(U1-GPIO7/ADC1_CH6-Pad7) -> /WA_SDA
- U1 pad 9: unconnected-(U1-GPIO16/ADC2_CH5/32K_N-Pad9) -> /SPARE_1
Routing:
- net +3V3: track 0.00 -> 174.3 mm
- net GND: track 0.00 -> 109.5 mm
- net /WA_BUSY: track 0.00 -> 58.8 mm
- net /WA_RESET: track 0.00 -> 55.0 mm
- net /WA_DC: track 0.00 -> 51.6 mm
- net /WA_SDA: track 0.00 -> 49.6 mm
- net /WA_CS: track 0.00 -> 47.1 mm
- net /WA_SCL: track 0.00 -> 42.5 mm
