File: docs/e-ink_multi_sensor/e-ink_multi_sensor/e-ink_multi_sensor.kicad_sch (KiCad schematic)
At the start: 0 parts

Commit message: documentation
Parts:
- added D1: WS2812B, LED_SMD:LED_WS2812B_PLCC4_5.0x5.0mm_P3.2mm, symbol LED:WS2812B
- added J1: HC-SR501, Sensor:Sensirion_SCD4x-1EP_10.1x10.1mm_P1.25mm_EP4.8x4.8mm, symbol Connector_Generic:Conn_01x03
- added U1: ESP32-S3-WROOM-1, RF_Module:ESP32-S3-WROOM-1, symbol RF_Module:ESP32-S3-WROOM-1
- added U2: BME280, Package_LGA:Bosch_LGA-8_2.5x2.5mm_P0.65mm_ClockwisePinNumbering, symbol Sensor:BME280
- added U3: SCD41-D-R2, Sensor:Sensirion_SCD4x-1EP_10.1x10.1mm_P1.25mm_EP4.8x4.8mm, symbol Sensor_Gas:SCD41-D-R2
Connections:
- new net +3V3: U1.2 (3V3), U2.2 (CSB), U2.5 (SDO), U2.6 (VDDIO), U2.8 (VDD), U3.19 (VDD), U3.7 (VDD)
- new net +5V: D1.1 (VDD), J1.1 (Pin_1)
- new net GND: D1.3 (VSS), J1.3 (Pin_3), U1.1 (GND), U1.40 (GND), U1.41 (GND), U2.1 (GND), U2.7 (GND), U3.20 (GND), U3.21 (GND), U3.6 (GND)
- new net I2C_SCL: U1.5 (IO5), U2.4 (SCK), U3.9 (SCL)
- new net I2C_SDA: U1.4 (IO4), U2.3 (SDI), U3.10 (SDA)
- new net PIR_GPIO12: J1.2 (Pin_2), U1.20 (IO12)

Commit message: schematic
Parts:
- removed U1: ESP32-S3-WROOM-1, RF_Module:ESP32-S3-WROOM-1, symbol RF_Module:ESP32-S3-WROOM-1
- removed U2: BME280, Package_LGA:Bosch_LGA-8_2.5x2.5mm_P0.65mm_ClockwisePinNumbering, symbol Sensor:BME280
- removed U3: SCD41-D-R2, Sensor:Sensirion_SCD4x-1EP_10.1x10.1mm_P1.25mm_EP4.8x4.8mm, symbol Sensor_Gas:SCD41-D-R2
- added J2: SCD41, PCM_Espressif:ESP32-S3-DevKitC, symbol Connector_Generic:Conn_01x04
- added J3: BME280, PCM_Espressif:ESP32-S3-DevKitC, symbol Connector_Generic:Conn_01x04
- added U1: ESP32-S3-DevKitC, PCM_Espressif:ESP32-S3-DevKitC, symbol PCM_Espressif:ESP32-S3-DevKitC
Connections:
- net +3V3: now also U1.1 (3V3), U1.2 (3V3)
- net GND: now also J2.4 (Pin_4), J3.4 (Pin_4), U1.22 (GND), U1.23 (GND), U1.24 (GND), U1.44 (GND)
- net I2C_SCL: now also J2.3 (Pin_3), J3.3 (Pin_3), U1.5 (GPIO5/ADC1_CH4)
- net I2C_SDA: now also J2.2 (Pin_2), J3.2 (Pin_2), U1.4 (GPIO4/ADC1_CH3)
- net PIR_GPIO12: now also U1.18 (GPIO12/ADC2_CH1)
- new net 3v3: J2.1 (Pin_1), J3.1 (Pin_1)
Other:
- note added: "BME280"
- note added: "SCD41"
- moved on the sheet: D1, J1

Commit message: schematic
Parts:
- J1: footprint Sensor:Sensirion_SCD4x-1EP_10.1x10.1mm_P1.25mm_EP4.8x4.8mm -> Connector_JST:JST_EH_B3B-EH-A_1x03_P2.50mm_Vertical
- J2, J3: footprint PCM_Espressif:ESP32-S3-DevKitC -> Connector:NS-Tech_Grove_1x04_P2mm_Vertical
Other:
- title: (none) -> Multi-sensor ESP32 board with e-ink display
- moved on the sheet: D1, J1, J2, J3, U1

Commit message: updated schematic
Parts:
- added H1, H2, H3, H4: MountingHole, MountingHole:MountingHole_3mm_Pad, symbol Mechanical:MountingHole
Other:
- note added: "Define pull-ups"

Commit message: added the WeAct e-ink display connector
Parts:
- added J4: WeAct, Connector_JST:JST_PH_B8B-PH-K_1x08_P2.00mm_Vertical, symbol Connector_Generic:Conn_01x08
Connections:
- net 3v3: now also J4.1 (Pin_1)
- net GND: now also J4.8 (Pin_8)
- new net WA_BUSY: J4.7 (Pin_7)
- new net WA_CS: J4.4 (Pin_4)
- new net WA_DC: J4.5 (Pin_5)
- new net WA_RST: J4.6 (Pin_6)
- new net WA_SPI_CLK: J4.2 (Pin_2)
- new net WA_SPI_MOSI: J4.3 (Pin_3)
Other:
- note added: "WeAct e-Ink"

Commit message: updated schematic
Parts:
- added J5: WeAct 2, Connector_Hirose:Hirose_DF11-8DP-2DSA_2x04_P2.00mm_Vertical, symbol Connector_Generic:Conn_02x04_Counter_Clockwise
- J4: value WeAct -> WeAct 1
Connections:
- net WA_RST is gone; now on net WA_SDA: J4.6 (Pin_6)
- net WA_SPI_CLK is gone; now on net WA_RESET: J4.2 (Pin_2)
- net WA_SPI_MOSI is gone; now on net WA_DC: J4.3 (Pin_3)
- net +3V3: now also J2.1 (Pin_1), J3.1 (Pin_1), J4.8 (Pin_8), J5.8 (Pin_8)
- net GND: now also J4.7 (Pin_7), J5.7 (Pin_7); no longer J4.8 (Pin_8)
- net I2C_SCL: no longer U1.5 (GPIO5/ADC1_CH4)
- net I2C_SDA: no longer U1.4 (GPIO4/ADC1_CH3)
- net PIR_GPIO12: no longer U1.18 (GPIO12/ADC2_CH1)
- net WA_BUSY: now also J4.1 (Pin_1), U1.17 (GPIO11/ADC2_CH0), J5.1 (Pin_1); no longer J4.7 (Pin_7)
- net WA_CS: now also U1.12 (GPIO8/ADC1_CH7), J5.4 (Pin_4)
- net WA_DC: now also U1.15 (GPIO9/ADC1_CH8), J5.3 (Pin_3); no longer J4.5 (Pin_5)
- net SPARE_2: now reaches U1.10 (GPIO17/ADC2_CH6)
- net SPARE_3: now reaches U1.11 (GPIO18/ADC2_CH7)
- net WA_RESET: now reaches U1.16 (GPIO10/ADC1_CH9)
- net WA_RESET: now also J5.2 (Pin_2)
- net SPARE_4: now reaches U1.27 (GPIO21)
- net WA_SCL: now reaches U1.6 (GPIO6/ADC1_CH5)
- net WA_SCL: now also J4.5 (Pin_5), J5.5 (Pin_5)
- net WA_SDA: now reaches U1.7 (GPIO7/ADC1_CH6)
- net WA_SDA: now also J5.6 (Pin_6)
- net SPARE_1: now reaches U1.9 (GPIO16/ADC2_CH5/32K_N)
- removed net 3v3: J2.1 (Pin_1), J3.1 (Pin_1), J4.1 (Pin_1)
Other:
- note removed: "BME280"
- note removed: "Define pull-ups"
- note removed: "SCD41"
- note removed: "WeAct e-Ink"
- moved on the sheet: J4
